Commit message: Changing structure of pal_hey5 gripper repo

File: pal_hey5_description/gazebo/gazebo.urdf.xacro (robot description, xacro)
@@ -17,5 +17,5 @@
    <xacro:property name="is_multiple" value="$(arg multiple)" />
    <xacro:property name="nsp" value="$(arg namespace)" />
-   <xacro:macro name="hey5_gazebo_simulation" params="side">
+   <xacro:macro name="pal_hey5_gazebo_simulation" params="side">
    <gazebo>
     <plugin filename="libgazebo_underactuated_finger.so" name="gazebo_${side}_thumb">

File: pal_hey5_description/robots/pal_hey5_test.urdf.xacro (robot description, xacro)
@@ -13,15 +13,15 @@
  -->
 <robot xmlns:xacro="http://ros.org/wiki/xacro"
-       name="hey5">
+       name="pal_hey5">
   <!--External resources-->
-  <xacro:include filename="$(find hey5_description)/urdf/deg_to_rad.urdf.xacro" />
-  <xacro:include filename="$(find hey5_description)/urdf/hey5_hand.urdf.xacro" />
+  <xacro:include filename="$(find pal_hey5_description)/urdf/deg_to_rad.urdf.xacro" />
+  <xacro:include filename="$(find pal_hey5_description)/urdf/pal_hey5_hand.urdf.xacro" />
   <!--Spawn hands-->
   <link name="tool_flange"/>
-  <xacro:hey5_hand parent="tool_flange" name="hand_right" reflect="1" >
+  <xacro:pal_hey5_hand parent="tool_flange" name="hand_right" reflect="1" >
     <origin xyz="0 0.13 0" rpy="0 ${-90 * deg_to_rad} ${90 * deg_to_rad}" />
-  </xacro:hey5_hand>
-  <xacro:hey5_hand parent="tool_flange" name="hand_left" reflect="-1" >
+  </xacro:pal_hey5_hand>
+  <xacro:pal_hey5_hand parent="tool_flange" name="hand_left" reflect="-1" >
     <origin xyz="0 -0.13 0" rpy="0 ${-90 * deg_to_rad} ${90 * deg_to_rad}" />
-  </xacro:hey5_hand>
+  </xacro:pal_hey5_hand>
 </robot>

File: pal_hey5_description/urdf/fingers.urdf.xacro (robot description, xacro)
@@ -14,6 +14,6 @@
 <robot xmlns:xacro="http://ros.org/wiki/xacro">
   <!--External resources-->
-  <xacro:include filename="$(find hey5_description)/urdf/deg_to_rad.urdf.xacro" />
-  <xacro:include filename="$(find hey5_description)/urdf/materials.urdf.xacro" />
+  <xacro:include filename="$(find pal_hey5_description)/urdf/deg_to_rad.urdf.xacro" />
+  <xacro:include filename="$(find pal_hey5_description)/urdf/materials.urdf.xacro" />
   <!--Constants-->
   <xacro:property name="thumb_abd_min"   value="${  0 * deg_to_rad}" />
@@ -125,12 +125,12 @@
         <origin xyz="0 0 0" rpy="0 0 0" />
         <geometry>
-          <mesh filename="package://hey5_description/meshes/finger_abd${vis_suffix}.stl" scale="1 1 ${reflect}" />
-        </geometry>
-        <material name="Hey5DarkGrey" />
-      </visual>
-      <collision>
-        <origin xyz="0 0 0" rpy="0 0 0" />
-        <geometry>
-          <mesh filename="package://hey5_description/meshes/finger_abd_collision.stl" scale="1 1 ${reflect}" />
+          <mesh filename="package://pal_hey5_description/meshes/finger_abd${vis_suffix}.stl" scale="1 1 ${reflect}" />
+        </geometry>
+        <material name="Hey5DarkGrey" />
+      </visual>
+      <collision>
+        <origin xyz="0 0 0" rpy="0 0 0" />
+        <geometry>
+          <mesh filename="package://pal_hey5_description/meshes/finger_abd_collision.stl" scale="1 1 ${reflect}" />
         </geometry>
       </collision>
@@ -166,12 +166,12 @@
         <origin xyz="0 0 0" rpy="0 0 0" />
         <geometry>
-          <mesh filename="package://hey5_description/meshes/thumb_abd${vis_suffix}.stl" scale="1 1 ${reflect}" />
-        </geometry>
-        <material name="Hey5DarkGrey" />
-      </visual>
-      <collision>
-        <origin xyz="0 0 0" rpy="0 0 0" />
-        <geometry>
-          <mesh filename="package://hey5_description/meshes/thumb_abd_collision.stl" scale="1 ${reflect} 1" />
+          <mesh filename="package://pal_hey5_description/meshes/thumb_abd${vis_suffix}.stl" scale="1 1 ${reflect}" />
+        </geometry>
+        <material name="Hey5DarkGrey" />
+      </visual>
+      <collision>
+        <origin xyz="0 0 0" rpy="0 0 0" />
+        <geometry>
+          <mesh filename="package://pal_hey5_description/meshes/thumb_abd_collision.stl" scale="1 ${reflect} 1" />
         </geometry>
       </collision>
@@ -251,12 +251,12 @@
         <origin xyz="0 0 0" rpy="0 0 0" />
         <geometry>
-          <mesh filename="package://hey5_description/meshes/finger_flex${vis_suffix}.stl" />
-        </geometry>
-        <material name="Hey5DarkGrey" />
-      </visual>
-      <collision>
-        <origin xyz="0 0 0" rpy="0 0 0" />
-        <geometry>
-          <mesh filename="package://hey5_description/meshes/finger_flex_collision.stl" />
+          <mesh filename="package://pal_hey5_description/meshes/finger_flex${vis_suffix}.stl" />
+        </geometry>
+        <material name="Hey5DarkGrey" />
+      </visual>
+      <collision>
+        <origin xyz="0 0 0" rpy="0 0 0" />
+        <geometry>
+          <mesh filename="package://pal_hey5_description/meshes/finger_flex_collision.stl" />
         </geometry>
       </collision>
@@ -294,12 +294,12 @@
         <origin xyz="0 0 0" rpy="0 0 0" />
         <geometry>
-          <mesh filename="package://hey5_description/meshes/finger_flex_tip${vis_suffix}.stl" />
-        </geometry>
-        <material name="Hey5DarkGrey" />
-      </visual>
-      <collision>
-        <origin xyz="0 0 0" rpy="0 0 0" />
-        <geometry>
-          <mesh filename="package://hey5_description/meshes/finger_flex_tip_collision.stl" />
+          <mesh filename="package://pal_hey5_description/meshes/finger_flex_tip${vis_suffix}.stl" />
+        </geometry>
+        <material name="Hey5DarkGrey" />
+      </visual>
+      <collision>
+        <origin xyz="0 0 0" rpy="0 0 0" />
+        <geometry>
+          <mesh filename="package://pal_hey5_description/meshes/finger_flex_tip_collision.stl" />
         </geometry>
       </collision>

File: pal_hey5_description/urdf/pal_hey5.ros2_control.xacro (robot description, xacro)
@@ -20,6 +20,6 @@
       <state_interface name="effort" />
     </joint>
-    <xacro:include filename="$(find hey5_description)/urdf/hey5.transmission.xacro" />
-    <xacro:hey5_simple_transmission name="${name}" reduction="${reduction}"/>
+    <xacro:include filename="$(find pal_hey5_description)/urdf/pal_hey5.transmission.xacro" />
+    <xacro:pal_hey5_simple_transmission name="${name}" reduction="${reduction}"/>
   </xacro:macro>
   <xacro:macro name="ros2_control_hey5" params="name" >

File: pal_hey5_description/urdf/pal_hey5.transmission.xacro (robot description, xacro)
@@ -13,5 +13,5 @@
  -->
 <robot xmlns:xacro="http://ros.org/wiki/xacro">
-  <xacro:macro name="hey5_simple_transmission" params="name reduction" >
+  <xacro:macro name="pal_hey5_simple_transmission" params="name reduction" >
     <transmission name="${name}_trans">
       <plugin>transmission_interface/SimpleTransmission</plugin>

File: pal_hey5_description/urdf/pal_hey5_hand.urdf.xacro (robot description, xacro)
@@ -14,10 +14,10 @@
 <robot xmlns:xacro="http://ros.org/wiki/xacro">
   <!--External resources-->
-  <xacro:include filename="$(find hey5_description)/urdf/actuators.urdf.xacro" />
-  <xacro:include filename="$(find hey5_description)/urdf/deg_to_rad.urdf.xacro" />
-  <xacro:include filename="$(find hey5_description)/urdf/fingers.urdf.xacro" />
-  <xacro:include filename="$(find hey5_description)/urdf/palm.urdf.xacro" />
-  <xacro:include filename="$(find hey5_description)/urdf/transmissions.urdf.xacro" />
-  <xacro:include filename="$(find hey5_description)/gazebo/gazebo.urdf.xacro" />
+  <xacro:include filename="$(find pal_hey5_description)/urdf/actuators.urdf.xacro" />
+  <xacro:include filename="$(find pal_hey5_description)/urdf/deg_to_rad.urdf.xacro" />
+  <xacro:include filename="$(find pal_hey5_description)/urdf/fingers.urdf.xacro" />
+  <xacro:include filename="$(find pal_hey5_description)/urdf/palm.urdf.xacro" />
+  <xacro:include filename="$(find pal_hey5_description)/urdf/transmissions.urdf.xacro" />
+  <xacro:include filename="$(find pal_hey5_description)/gazebo/gazebo.urdf.xacro" />
   <!--Constants-->
   <xacro:property name="thumb_act_flex_start"  value="2.0" />
@@ -34,5 +34,5 @@
     - origin: XML block containing the pose of the palm link with respect to its parent
   -->
-  <xacro:macro name="hey5_hand" params="name parent reflect *origin">
+  <xacro:macro name="pal_hey5_hand" params="name parent reflect *origin">
   <!-- Tool Link -->
     <link name="${name}_tool_link">
@@ -135,6 +135,6 @@
       <origin xyz="0.13 0.02 0" rpy="0 0 0"/>
     </joint>
-    <!-- hey5 gazebo plugin -->
-    <xacro:hey5_gazebo_simulation side="${name}"/>
+    <!-- pal_hey5 gazebo plugin -->
+    <xacro:pal_hey5_gazebo_simulation side="${name}"/>
   </xacro:macro>
 </robot>

File: pal_hey5_description/urdf/palm.urdf.xacro (robot description, xacro)
@@ -37,5 +37,5 @@
         <origin xyz="0 0 0" rpy="0 0 0" />
         <geometry>
-          <mesh filename="package://hey5_description/meshes/palm.stl" scale="1 1 ${reflect}" />
+          <mesh filename="package://pal_hey5_description/meshes/palm.stl" scale="1 1 ${reflect}" />
         </geometry>
         <material name="Hey5DarkGrey" />
@@ -44,5 +44,5 @@
         <origin xyz="0 0 0" rpy="0 0 0" />
         <geometry>
-          <mesh filename="package://hey5_description/meshes/palm_collision.stl" scale="1 1 ${reflect}" />
+          <mesh filename="package://pal_hey5_description/meshes/palm_collision.stl" scale="1 1 ${reflect}" />
         </geometry>
       </collision>

File: pal_hey5_description/urdf/transmissions.urdf.xacro (robot description, xacro)
@@ -14,5 +14,5 @@
 <robot xmlns:xacro="http://ros.org/wiki/xacro">
   <!--External resources-->
-  <xacro:include filename="$(find hey5_description)/urdf/deg_to_rad.urdf.xacro" />
+  <xacro:include filename="$(find pal_hey5_description)/urdf/deg_to_rad.urdf.xacro" />
   <!--
     Specify transmissions for the thumb finger.
