Commit message: Use pal_urdf_utils materials and deg_to_rad

File: pal_hey5_description/robots/pal_hey5_test.urdf.xacro (robot description, xacro)
@@ -15,5 +15,5 @@
        name="pal_hey5">
   <!--External resources-->
-  <xacro:include filename="$(find pal_hey5_description)/urdf/deg_to_rad.urdf.xacro" />
+  <xacro:include filename="$(find pal_urdf_utils)/urdf/deg_to_rad.urdf.xacro" />
   <xacro:include filename="$(find pal_hey5_description)/urdf/pal_hey5_hand.urdf.xacro" />
   <!--Spawn hands-->

File: pal_hey5_description/urdf/actuators.urdf.xacro (robot description, xacro)
@@ -76,5 +76,5 @@
           <sphere radius="0.001"/>
         </geometry>
-        <material name="Hey5DarkGrey" />
+        <material name="DarkGrey" />
       </visual>
       <collision>

File: pal_hey5_description/urdf/fingers.urdf.xacro (robot description, xacro)
@@ -14,6 +14,6 @@
 <robot xmlns:xacro="http://ros.org/wiki/xacro">
   <!--External resources-->
-  <xacro:include filename="$(find pal_hey5_description)/urdf/deg_to_rad.urdf.xacro" />
-  <xacro:include filename="$(find pal_hey5_description)/urdf/materials.urdf.xacro" />
+  <xacro:include filename="$(find pal_urdf_utils)/urdf/deg_to_rad.urdf.xacro" />
+  <xacro:include filename="$(find pal_urdf_utils)/urdf/materials.urdf.xacro" />
   <!--Constants-->
   <xacro:property name="thumb_abd_min"   value="${  0 * deg_to_rad}" />
@@ -127,5 +127,5 @@
           <mesh filename="package://pal_hey5_description/meshes/finger_abd${vis_suffix}.stl" scale="1 1 ${reflect}" />
         </geometry>
-        <material name="Hey5DarkGrey" />
+        <material name="DarkGrey" />
       </visual>
       <collision>
@@ -168,5 +168,5 @@
           <mesh filename="package://pal_hey5_description/meshes/thumb_abd${vis_suffix}.stl" scale="1 1 ${reflect}" />
         </geometry>
-        <material name="Hey5DarkGrey" />
+        <material name="DarkGrey" />
       </visual>
       <collision>
@@ -210,5 +210,5 @@
           <box size="${finger_d2} 0.002 0.012" />
         </geometry>
-        <material name="Hey5DarkGrey" />
+        <material name="DarkGrey" />
       </visual>
       <collision>
@@ -253,5 +253,5 @@
           <mesh filename="package://pal_hey5_description/meshes/finger_flex${vis_suffix}.stl" />
         </geometry>
-        <material name="Hey5DarkGrey" />
+        <material name="DarkGrey" />
       </visual>
       <collision>
@@ -296,5 +296,5 @@
           <mesh filename="package://pal_hey5_description/meshes/finger_flex_tip${vis_suffix}.stl" />
         </geometry>
-        <material name="Hey5DarkGrey" />
+        <material name="DarkGrey" />
       </visual>
       <collision>

File: pal_hey5_description/urdf/pal_hey5_hand.urdf.xacro (robot description, xacro)
@@ -15,5 +15,5 @@
   <!--External resources-->
   <xacro:include filename="$(find pal_hey5_description)/urdf/actuators.urdf.xacro" />
-  <xacro:include filename="$(find pal_hey5_description)/urdf/deg_to_rad.urdf.xacro" />
+  <xacro:include filename="$(find pal_urdf_utils)/urdf/deg_to_rad.urdf.xacro" />
   <xacro:include filename="$(find pal_hey5_description)/urdf/fingers.urdf.xacro" />
   <xacro:include filename="$(find pal_hey5_description)/urdf/palm.urdf.xacro" />

File: pal_hey5_description/urdf/palm.urdf.xacro (robot description, xacro)
@@ -39,5 +39,5 @@
           <mesh filename="package://pal_hey5_description/meshes/palm.stl" scale="1 1 ${reflect}" />
         </geometry>
-        <material name="Hey5DarkGrey" />
+        <material name="DarkGrey" />
       </visual>
       <collision>

File: pal_hey5_description/urdf/transmissions.urdf.xacro (robot description, xacro)
@@ -14,5 +14,5 @@
 <robot xmlns:xacro="http://ros.org/wiki/xacro">
   <!--External resources-->
-  <xacro:include filename="$(find pal_hey5_description)/urdf/deg_to_rad.urdf.xacro" />
+  <xacro:include filename="$(find pal_urdf_utils)/urdf/deg_to_rad.urdf.xacro" />
   <!--
     Specify transmissions for the thumb finger.
