Commit message: remove and fix wrong inertia

File: pal_hey5_description/urdf/actuators.urdf.xacro (robot description, xacro)
@@ -65,24 +65,5 @@
       <xacro:insert_block name="safety_controller" />
     </joint>
-    <link name="${name}_link">
-      <inertial>
-        <origin xyz="0 0 0" rpy="0 0 0" />
-        <mass value="0.05" />
-        <inertia ixx="0.001" ixy="0" ixz="0" iyy="0.001" iyz="0" izz="0.001" /> <!--To stabilize simulation-->
-      </inertial>
-      <visual>
-        <origin xyz="0 0 0" rpy="0 0 0" />
-        <geometry>
-          <sphere radius="0.001"/>
-        </geometry>
-        <material name="DarkGrey" />
-      </visual>
-      <collision>
-        <origin xyz="0 0 0" rpy="0 0 0" />
-        <geometry>
-          <sphere radius="0.001"/>
-        </geometry>
-      </collision>
-    </link>
+    <link name="${name}_link"/>
   </xacro:macro>
 </robot>

File: pal_hey5_description/urdf/pal_hey5_hand.urdf.xacro (robot description, xacro)
@@ -36,13 +36,5 @@
   <xacro:macro name="pal_hey5_hand" params="name parent reflect *origin">
   <!-- Tool Link -->
-    <link name="${name}_tool_link">
-      <inertial>
-        <origin xyz="0 0 0" rpy="0 0 0" />
-        <mass value="0.0001" />
-        <inertia ixx="0.00001" ixy="0.0" ixz="0.0"
-                 iyy="0.00001" iyz="0.0"
-                 izz="0.00001" />
-      </inertial>
-    </link>
+    <link name="${name}_tool_link"/>
     <joint name="${name}_tool_joint" type="fixed">
       <xacro:insert_block name="origin"/>
